Commit message: Added four wheel joints and update robot dimensions

File: urdf/autonomous_robot.urdf (robot description, URDF)
Before this commit: robot autonomous_robot, 5 links, 0 joints
Links:
- link left_rear_wheel: geometry visual cylinder length=0.025 radius=0.05
- link right_front_wheel: geometry visual cylinder length=0.025 radius=0.05
- link right_rear_wheel: geometry visual cylinder length=0.025 radius=0.05
Joints:
- added joint left_front_wheel_joint: type continuous, parent base_link, child left_front_wheel, origin xyz=0.10 0.115 0 rpy=1.5708 0 0, axis 0 0 1
- added joint left_rear_wheel_joint: type continuous, parent base_link, child left_rear_wheel, origin xyz=-0.10 0.115 0 rpy=1.5708 0 0, axis 0 0 1
- added joint right_front_wheel_joint: type continuous, parent base_link, child right_front_wheel, origin xyz=0.10 -0.115 0 rpy=1.5708 0 0, axis 0 0 1
- added joint right_rear_wheel_joint: type continuous, parent base_link, child right_rear_wheel, origin xyz=-0.10 -0.115 0 rpy=1.5708 0 0, axis 0 0 1
